File: ReadVRAM.kicad_sch (KiCad schematic)
At the start: 3 parts, among them U2 IDT7202, U3 GAL22V10, U4 IDT7007

Commit message: starting to work on VRAM module design
Parts:
- removed U2: IDT7202, symbol Memory_RAM:IDT7202
- removed U4: IDT7007, MODULE, symbol IDT7007:IDT7007
- renumbered U3 to U701
