File: HardwareDesign/Readout.kicad_sch (KiCad schematic)
At the start: 12 parts, among them U701 74ACT163, U702 74ACT163, U703 74ACT163, U705 74ACT273, U706 74ACT273, U707 GAL22V10

Commit message: use 74ALS163 rather than 74ACT163
The prototype did not work reliably with 74ACT163 counters,
but did work correctly with 74ALS163 counters.
Parts:
- U701, U702, U703: value 74ACT163 -> 74ALS163
Changed lines of the file:
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@@
 			)
 		)
-		(property "Value" "74ACT163"
+		(property "Value" "74ALS163"
 			(at 129.1941 132.08 0)
 			(effects
@@
 			)
 		)
-		(property "Value" "74ACT163"
+		(property "Value" "74ALS163"
 			(at 197.7741 132.08 0)
 			(effects
@@
 			)
 		)
-		(property "Value" "74ACT163"
+		(property "Value" "74ALS163"
 			(at 65.6941 132.08 0)
 			(effects

Commit message: use 74ALS and 74HCT parts where possible
The '574 implementing the VRAM module's bank register
can be a 74HCT574 because it's only driven by
(relatively slow) signals from the host system.

Changed the Readout module to use 74ALS273 rather than
74ACT273 for the row begin address register.

Changed the Pixgen module to use 74ALS574 rather than
74ACT574 for the character and attribute registers.
Parts:
- U705, U706: value 74ACT273 -> 74ALS273
Changed lines of the file:
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@@
 			)
 		)
-		(property "Value" "74ACT273"
+		(property "Value" "74ALS273"
 			(at 242.2241 39.37 0)
 			(effects
@@
 			)
 		)
-		(property "Value" "74ACT273"
+		(property "Value" "74ALS273"
 			(at 174.9141 39.37 0)
 			(effects
