File: HardwareDesign/Pixgen.kicad_sch (KiCad schematic)
At the start: 11 parts, among them U601 GAL22V10, U602 74ALS574, U603 27SF512, U604 74ALS574, U605 GAL22V10

Commit message: pixel generator works better with 74ACT574
With 74ALS574 parts for the character and attribute
register, we were getting some minor display artifacts.
Parts:
- U602, U604: value 74ALS574 -> 74ACT574
Changed lines of the file:
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@@
 			)
 		)
-		(property "Value" "74ALS574"
+		(property "Value" "74ACT574"
 			(at 79.6641 59.69 0)
 			(effects
@@
 			)
 		)
-		(property "Value" "74ALS574"
+		(property "Value" "74ACT574"
 			(at 65.6941 119.38 0)
 			(effects
