File: HardwareDesign/HW_VGA.kicad_sch (KiCad schematic)
At the start: 6 parts, among them J1 Conn_02x40_Odd_Even, J401 Conn_01x06, U1 25.175 MHz, U301 GAL22V10

Commit message: use jumper to connect VRefresh to IRQ6
I'm not 100% certain this feature will work (it doesn't
on the prototype), so the jumper allows it to be
selectively enable or disabled.
Parts:
- added J301: Conn_01x02, symbol Connector_Generic:Conn_01x02
Connections:
- net IRQ6: now also J301.2 (Pin_2); no longer U301.20 (I/O18)
- new net VRefresh: J301.1 (Pin_1), U301.20 (I/O18)
Other:
- note added: "Experimental: place jumper to generate a vertical refresh interrupt as IRQ6"
- note removed: "Note that pin 20 is a one-cycle vertical refresh pulse, which is sent to the interrupt controller as the edge-triggered IRQ6."
Changed lines of the file:
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@@
 	(wire
 		(pts
+			(xy 306.07 59.69) (xy 321.31 59.69)
+		)
+		(stroke
+			(width 0)
+			(type default)
+		)
+	)
+	(wire
+		(pts
 			(xy 53.34 156.21) (xy 67.31 156.21)
 		)
@@
 	(wire
 		(pts
-			(xy 279.4 59.69) (xy 297.18 59.69)
+			(xy 279.4 59.69) (xy 303.53 59.69)
 		)
 		(stroke
@@
 		)
 	)
-	(text "Note that pin 20 is a one-cycle\nvertical refresh pulse, which is\nsent to the interrupt controller\nas the edge-triggered IRQ6."
-		(exclude_from_sim no)
-		(at 304.8 51.054 0)
-		(effects
-			(font
-				(size 1.27 1.27)
-			)
-		)
-	)
 	(text "Sync gen and visibility signals:\nLogic is in Sync.pld"
 		(exclude_from_sim no)
@@
 		)
 	)
+	(text "Experimental: place jumper\nto generate a vertical\nrefresh interrupt as IRQ6"
+		(exclude_from_sim no)
+		(at 308.864 48.768 0)
+		(effects
+			(font
+				(size 1.27 1.27)
+			)
+		)
+	)
 	(text "Horizontal count"
 		(exclude_from_sim no)
@@
 	)
 	(label "IRQ6"
-		(at 281.94 59.69 0)
+		(at 314.96 59.69 0)
 		(fields_autoplaced yes)
 		(effects
@@
 		)
 	)
+	(label "VRefresh"
+		(at 281.94 59.69 0)
+		(fields_autoplaced yes)
+		(effects
+			(font
+				(size 1.27 1.27)
+			)
+			(justify left bottom)
+		)
+	)
 	(label "PC6"
 		(at 29.21 130.81 0)
@@
 					(unit 1)
 				)
+			)
+		)
+	)
+	(symbol
+		(lib_id "Connector_Generic:Conn_01x02")
+		(at 303.53 54.61 90)
+		(unit 1)
+		(exclude_from_sim no)
+		(in_bom yes)
+		(on_board yes)
+		(dnp no)
+		(fields_autoplaced yes)
+		(property "Reference" "J301"
+			(at 308.61 53.3399 90)
+			(effects
+				(font
+					(size 1.27 1.27)
+				)
+				(justify right)
+			)
+		)
+		(property "Value" "Conn_01x02"
+			(at 308.61 55.8799 90)
+			(effects
+				(font
+					(size 1.27 1.27)
+				)
+				(justify right)
+			)
+		)
+		(property "Footprint" ""
+			(at 303.53 54.61 0)
+			(effects
+				(font
+					(size 1.27 1.27)
+				)
+				(hide yes)
+			)
+		)
+		(property "Datasheet" "~"
+			(at 303.53 54.61 0)
+			(effects
+				(font
+					(size 1.27 1.27)
+				)
+				(hide yes)
+			)
+		)
+		(property "Description" "Generic connector, single row, 01x02, script generated (kicad-library-utils/schlib/autogen/connector/)"
+			(at 303.53 54.61 0)
+			(effects
+				(font
+					(size 1.27 1.27)
+				)
+				(hide yes)
+			)
+		)
+		(pin "1"
+		)
+		(pin "2"
+		)
+		(instances
+			(project ""
+				(path "/c4bd4b39-993a-4195-805f-b4de6fa4aea5"
+					(reference "J301")
+					(unit 1)
+				)
